Commit message: [change] file locations

File: urdf/models/kinect.urdf (robot description, URDF)
Before this commit: robot camera, 3 links, 2 joints
Links:
- link kinect_link: geometry collision box size=0.065 0.25 0.082; visual mesh filename=package://kinect_bringup/urdf/meshes/kinectv2.stl

File: urdf/sensor/kinect.urdf.xacro (robot description, xacro)
@@ -6,5 +6,5 @@
 		<material name="black"/>
         <geometry>
-          <mesh filename="package://kinect_bringup/meshes/kinectv2.stl"/>
+          <mesh filename="package://kinect_bringup/urdf/meshes/kinectv2.stl"/>
         </geometry>
       </visual>
